File: brain.brd (EAGLE design)
At the start: 100.1 x 80 mm, 24 parts, among them IC1 LP2950ACZ-3.3, IC2 LP2950ACZ-3.3, U1 TINY45-20-DIP, U4 TINY45-20-DIP, U5 TINY45-20-DIP, U6 TINY45-20-DIP

Commit message: Added bypass capacitors per Sasha's request. Put some identifying information on bottom silkscreen.
Parts:
- added C10, C7, C8, C9: bypass, rcl:C050-025X075
Connections:
- net GND1: now also C10.2, C7.2
- net GND2: now also C8.2, C9.2
- net VCC1: now also C10.1, C7.1
- net VOUT2: now also C8.1, C9.1
Routing:
- net PB11: track 77.5 -> 32.7 mm
- net GND1: track 146.6 -> 172.8 mm
- net VOUT2: track 88.4 -> 111.3 mm
- net N$6: track 13.8 -> 0.00 mm
- net N$15: track 0.00 -> 13.4 mm
- net VCC1: track 107.3 -> 119.3 mm, vias 0 -> 1
- net GND2: track 141.4 -> 150.9 mm
- net N$10: track 0.00 -> 8.42 mm
- net N$12: track 0.00 -> 7.48 mm
Other:
- board size 100.1 x 80 mm -> 100 x 80.3 mm
- board text added: "Felipe Vargas Robert Viramontes Jessica Zhao"
- board text added: "Receiver"
- board text added: "Transmitter"
- board text added: "Well Monitoring System"
